File: PCB/PCB.sch (KiCad schematic (older format))
At the start: 35 parts

Commit message: Update PCB.sch
Parts:
- removed R?: R, symbol Device:R
- added C? (x5): C, symbol Device:C
- added D?: LED_ALT, symbol Device:LED_ALT
- added D? (x8): D_Sch, symbol Device:D_Schottky
- added J?: Conn_01x02_Female, symbol Connector:Conn_01x02_Female
- added Q? (x7): Q-NPN, symbol Device:Q_NPN_BCE
- added Q? (x5): Q-PNP, symbol Device:Q_PNP_BCE
- added R? (x26): R, symbol Device:R
Connections:
- net GND: now also J?.2 (Pin_2), R?.1, R?.2
- net VCC: now also C?.2, Q?.2 (C), Q?.2 (C)
- net VEE: now also C?.1, D?.1 (K), Q?.2 (C), Q?.2 (C)
- net at D?.1 (K): now also D?.2 (A)
- net at Q?.1 (B), Q?.2 (C), Q?.3 (E)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: now also C?.1
- net at C?.2, Q?.1 (B), Q?.2 (C)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: now also C?.2
- net at Q?.3 (E): now also Q?.3 (E), Q?.3 (E) (x2)
- net at Q?.1 (B): now also D?.2 (A)
- net at Q?.2 (C): now also Q?.1 (B), R?.1, R?.1
- net at Q?.2 (C): now also R?.1
- new net: C?.1, Q?.1 (B), R?.2
- new net: Q?.3 (E), R?.2, R?.2, R?.2
- new net: Q?.1 (B), R?.1, R?.2 (x2)
- new net: D?.1 (K), Q?.2 (C), R?.2
- new net: C?.2, D?.1 (K), R?.1
- new net: D?.1 (K), R?.1
- new net: C?.1, R?.1
- new net: D?.2 (A), Q?.2 (C)
- new net: Q?.1 (B), R?.1 (x2)
- new net: D?.1 (K), Q?.3 (E)
- new net: D?.2 (A), R?.2
- new net: R?.1, R?.1, R?.1, R?.2
- new net: D?.1 (K), D?.2 (A), J?.1 (Pin_1), R?.1, R?.1, R?.2, R?.2
- new net: Q?.1 (B), Q?.3 (E), R?.1
- new net: Q?.3 (E), Q?.3 (E), R?.1
- new net: Q?.1 (B), R?.2 (x2)
- new net: Q?.1 (B), Q?.2 (C), R?.1, R?.2
- new net: D?.2 (A), Q?.2 (C), R?.1, R?.2
- new net: D?.1 (K), Q?.1 (B)
- new net: Q?.3 (E), R?.1, R?.1, R?.1
- new net: Q?.2 (C), R?.1, R?.2
- new net: C?.1, D?.2 (A), R?.2
- new net: C?.2, R?.2
- new net: D?.1 (K), Q?.2 (C)
- new net: D?.2 (A), Q?.3 (E)
- new net: D?.1 (K), R?.1, R?.2, R?.2
- new net: D?.2 (A), R?.1
- new net: C?.2, Q?.1 (B), R?.2
- new net: Q?.1 (B), Q?.3 (E), R?.2
- new net: Q?.3 (E), Q?.3 (E), R?.2
- new net +15V: Q?.2 (C), R?.2
- new net -15V: Q?.2 (C), R?.2
Other:
- moved on the sheet: Q?

Commit message: Update PCB.sch
Parts:
- added J?: Conn, symbol Connector:Conn_01x02_Female
- J?: value Conn_01x02_Female -> Conn
Connections:
- net GND: now also J?.2 (Pin_2)
- net at C?.1: now also J?.1 (Pin_1)
Other:
- moved on the sheet: C?, R?
Changed lines of the file:
@@
 L power:GND #PWR?
 U 1 1 5D17CE43
-P 1250 5250
-F 0 "#PWR?" H 1250 5000 50  0001 C CNN
-F 1 "GND" H 1255 5077 50  0000 C CNN
-F 2 "" H 1250 5250 50  0001 C CNN
-F 3 "" H 1250 5250 50  0001 C CNN
-	1    1250 5250
+P 1300 5250
+F 0 "#PWR?" H 1300 5000 50  0001 C CNN
+F 1 "GND" H 1305 5077 50  0000 C CNN
+F 2 "" H 1300 5250 50  0001 C CNN
+F 3 "" H 1300 5250 50  0001 C CNN
+	1    1300 5250
 	1    0    0    -1
 $EndComp
@@
 L Device:R R?
 U 1 1 5D23111A
-P 1250 4900
-F 0 "R?" H 1320 4946 50  0000 L CNN
-F 1 "R" H 1320 4855 50  0000 L CNN
-F 2 "" V 1180 4900 50  0001 C CNN
-F 3 "~" H 1250 4900 50  0001 C CNN
-	1    1250 4900
-	1    0    0    -1
-$EndComp
-Wire Wire Line
-	1250 4550 1250 4750
-Wire Wire Line
-	1250 5050 1250 5250
+P 1300 4900
+F 0 "R?" H 1370 4946 50  0000 L CNN
+F 1 "R" H 1370 4855 50  0000 L CNN
+F 2 "" V 1230 4900 50  0001 C CNN
+F 3 "~" H 1300 4900 50  0001 C CNN
+	1    1300 4900
+	1    0    0    -1
+$EndComp
 $Comp
 L Device:C C?
 U 1 1 5D239A3E
-P 1000 4550
-F 0 "C?" V 1252 4550 50  0000 C CNN
-F 1 "C" V 1161 4550 50  0000 C CNN
-F 2 "" H 1038 4400 50  0001 C CNN
-F 3 "~" H 1000 4550 50  0001 C CNN
-	1    1000 4550
-	0    -1   -1   0
-$EndComp
-Wire Wire Line
-	1150 4550 1250 4550
-Wire Wire Line
-	1350 4550 1250 4550
-Connection ~ 1250 4550
+P 1100 4550
+F 0 "C?" V 1352 4550 50  0000 C CNN
+F 1 "C" V 1261 4550 50  0000 C CNN
+F 2 "" H 1138 4400 50  0001 C CNN
+F 3 "~" H 1100 4550 50  0001 C CNN
+	1    1100 4550
+	0    -1   -1   0
+$EndComp
 Wire Wire Line
 	3250 5850 3950 5850
@@
 P 10550 3350
 F 0 "J?" H 10578 3326 50  0000 L CNN
-F 1 "Conn_01x02_Female" H 10578 3235 50  0000 L CNN
+F 1 "Conn" H 10578 3235 50  0000 L CNN
 F 2 "" H 10550 3350 50  0001 C CNN
 F 3 "~" H 10550 3350 50  0001 C CNN
@@
 Wire Wire Line
 	9950 4000 9950 5600
+$Comp
+L Connector:Conn_01x02_Female J?
+U 1 1 5D1D8FF0
+P 650 4550
+F 0 "J?" H 542 4735 50  0000 C CNN
+F 1 "Conn" H 542 4644 50  0000 C CNN
+F 2 "" H 650 4550 50  0001 C CNN
+F 3 "~" H 650 4550 50  0001 C CNN
+	1    650  4550
+	-1   0    0    -1
+$EndComp
+Wire Wire Line
+	1300 5250 1300 5150
+Wire Wire Line
+	1300 4750 1300 4550
+Wire Wire Line
+	1300 4550 1250 4550
+Wire Wire Line
+	1350 4550 1300 4550
+Connection ~ 1300 4550
+Wire Wire Line
+	850  4550 950  4550
+Wire Wire Line
+	850  4650 950  4650
+Wire Wire Line
+	950  4650 950  5150
+Wire Wire Line
+	950  5150 1300 5150
+Connection ~ 1300 5150
+Wire Wire Line
+	1300 5150 1300 5050
 $EndSCHEMATC

Commit message: gato
Parts:
- added C10: C, Capacitor_SMD:C_0805_2012Metric_Pad1.15x1.40mm_HandSolder, symbol Device:C
- added R41: R, Resistor_SMD:R_0805_2012Metric_Pad1.15x1.40mm_HandSolder, symbol Device:R
- C1, C5: renamed from C?; footprint (none) -> Capacitor_SMD:C_0603_1608Metric_Pad1.05x0.95mm_HandSolder
- C2: renamed from C?; footprint (none) -> Capacitor_THT:CP_Axial_L29.0mm_D16.0mm_P35.00mm_Horizontal
- C3, C4: renamed from C?; footprint (none) -> Capacitor_SMD:C_0805_2012Metric_Pad1.15x1.40mm_HandSolder
- C6, C7, C8, C9: renamed from C?; footprint (none) -> Capacitor_SMD:C_1206_3216Metric_Pad1.42x1.75mm_HandSolder
- D1, D2: renamed from D?; footprint (none) -> LED_THT:LED_D5.0mm
- D10, D3, D4, D5, D6, D7, D8, D9: renamed from D?; footprint (none) -> Diode_THT:D_DO-27_P5.08mm_Vertical_AnodeUp
- J1, J2: renamed from J?; footprint (none) -> Connector:Banana_Jack_2Pin
- Q1, Q11, Q14, Q15, Q16, Q17, Q18, Q19, Q2, Q20, Q21, Q3, Q4, Q5, Q6, Q7, Q9: renamed from Q?; footprint (none) -> Package_TO_SOT_SMD:SOT-23_Handsoldering
- Q10, Q12: renamed from Q?; value Q_NPN_BCE -> Q_NPN; footprint (none) -> Package_TO_SOT_SMD:SOT-23_Handsoldering
- Q13: renamed from Q?; value Q_PNP_BCE -> Q_PNP; footprint (none) -> Package_TO_SOT_SMD:SOT-23_Handsoldering
- Q22, Q23, Q24, Q25, Q26, Q27, Q8: renamed from Q?; footprint (none) -> Package_TO_SOT_THT:TO-3P-3_Horizontal_TabDown
- R1, R10, R11, R12, R13, R14, R15, R16, R17, R18, R19, R2, R20, R21, R22, R23, R24, R25, R26, R27, R28, R29, R3, R30, R31, R32, R33, R34, R35, R36, R37, R38, R39, R4, R40, R5, R6, R7, R8, R9: renamed from R?; footprint (none) -> Resistor_SMD:R_0805_2012Metric_Pad1.15x1.40mm_HandSolder
Connections:
- net +15V: now also D10.1 (K), D9.2 (A), J2.1 (Pin_1), R37.2, R38.1, R39.2, R40.1, C10.2, R41.1
- net at Q5.1 (B), R9.1: now also C10.1, R41.2
Other:
- moved on the sheet: C6, D10, D4, D6, D7, J2, Q10, Q12, Q16, Q19, Q20, Q23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

Commit message: pcb
Parts:
- C2: footprint Capacitor_THT:CP_Axial_L29.0mm_D16.0mm_P35.00mm_Horizontal -> Capacitor_THT:CP_Axial_L11.0mm_D5.0mm_P18.00mm_Horizontal
- D10, D3, D4, D5, D6, D7, D8, D9: footprint Diode_THT:D_DO-27_P5.08mm_Vertical_AnodeUp -> Diode_SMD:D_SOT-23_ANK
- J1: footprint Connector:Banana_Jack_2Pin -> Connector_Audio:Jack_3.5mm_CUI_SJ1-3533NG_Horizontal_CircularHoles
- J2: footprint Connector:Banana_Jack_2Pin -> Connector:JWT_A3963_1x02_P3.96mm_Vertical
- Q24, Q25: footprint Package_TO_SOT_THT:TO-3P-3_Horizontal_TabDown -> Package_TO_SOT_SMD:SOT-23_Handsoldering
- R39, R40: footprint Resistor_SMD:R_0805_2012Metric_Pad1.15x1.40mm_HandSolder -> Resistor_THT:R_Axial_Power_L25.0mm_W9.0mm_P30.48mm
Connections:
- net +15V: no longer C10.2, D10.1 (K), D9.2 (A), J2.1 (Pin_1), R37.2, R38.1, R39.2, R40.1, R41.1
- new net: C10.2, D10.1 (K), D9.2 (A), J2.1 (Pin_1), R37.2, R38.1, R39.2, R40.1, R41.1
Changed lines of the file:
@@
 F 0 "C2" H 3085 5054 50  0000 R CNN
 F 1 "C" H 3085 5145 50  0000 R CNN
-F 2 "Capacitor_THT:CP_Axial_L29.0mm_D16.0mm_P35.00mm_Horizontal" H 3238 4950 50  0001 C CNN
+F 2 "Capacitor_THT:CP_Axial_L11.0mm_D5.0mm_P18.00mm_Horizontal" H 3238 4950 50  0001 C CNN
 F 3 "~" H 3200 5100 50  0001 C CNN
 	1    3200 5100
@@
 F 0 "D3" V 6546 1421 50  0000 R CNN
 F 1 "D_Sch" V 6455 1421 50  0000 R CNN
-F 2 "Diode_THT:D_DO-27_P5.08mm_Vertical_AnodeUp" H 6500 1500 50  0001 C CNN
+F 2 "Diode_SMD:D_SOT-23_ANK" H 6500 1500 50  0001 C CNN
 F 3 "~" H 6500 1500 50  0001 C CNN
 	1    6500 1500
@@
 F 0 "D9" H 8050 1134 50  0000 C CNN
 F 1 "D_Sch" H 8050 1225 50  0000 C CNN
-F 2 "Diode_THT:D_DO-27_P5.08mm_Vertical_AnodeUp" H 8050 1350 50  0001 C CNN
+F 2 "Diode_SMD:D_SOT-23_ANK" H 8050 1350 50  0001 C CNN
 F 3 "~" H 8050 1350 50  0001 C CNN
 	1    8050 1350
@@
 F 0 "D5" V 7246 2271 50  0000 R CNN
 F 1 "D_Sch" V 7155 2271 50  0000 R CNN
-F 2 "Diode_THT:D_DO-27_P5.08mm_Vertical_AnodeUp" H 7200 2350 50  0001 C CNN
+F 2 "Diode_SMD:D_SOT-23_ANK" H 7200 2350 50  0001 C CNN
 F 3 "~" H 7200 2350 50  0001 C CNN
 	1    7200 2350
@@
 F 0 "D8" V 7846 2271 50  0000 R CNN
 F 1 "D_Sch" V 7755 2271 50  0000 R CNN
-F 2 "Diode_THT:D_DO-27_P5.08mm_Vertical_AnodeUp" H 7800 2350 50  0001 C CNN
+F 2 "Diode_SMD:D_SOT-23_ANK" H 7800 2350 50  0001 C CNN
 F 3 "~" H 7800 2350 50  0001 C CNN
 	1    7800 2350
@@
 F 0 "Q25" H 9641 1096 50  0000 L CNN
 F 1 "Q-NPN" H 9641 1005 50  0000 L CNN
-F 2 "Package_TO_SOT_THT:TO-3P-3_Horizontal_TabDown" H 9650 1150 50  0001 C CNN
+F 2 "Package_TO_SOT_SMD:SOT-23_Handsoldering" H 9650 1150 50  0001 C CNN
 F 3 "~" H 9450 1050 50  0001 C CNN
 	1    9450 1050
@@
 	9650 1350 9550 1350
 Wire Wire Line
-	8950 1850 9050 1850
-Wire Wire Line
 	9650 2750 9650 1350
 Connection ~ 9650 1350
@@
 F 0 "R39" H 10020 2946 50  0000 L CNN
 F 1 "R" H 10020 2855 50  0000 L CNN
-F 2 "Resistor_SMD:R_0805_2012Metric_Pad1.15x1.40mm_HandSolder" V 9880 2900 50  0001 C CNN
+F 2 "Resistor_THT:R_Axial_Power_L25.0mm_W9.0mm_P30.48mm" V 9880 2900 50  0001 C CNN
 F 3 "~" H 9950 2900 50  0001 C CNN
 	1    9950 2900
@@
 F 0 "J2" H 10578 3476 50  0000 L CNN
 F 1 "Conn" H 10578 3385 50  0000 L CNN
-F 2 "Connector:Banana_Jack_2Pin" H 10550 3500 50  0001 C CNN
+F 2 "Connector:JWT_A3963_1x02_P3.96mm_Vertical" H 10550 3500 50  0001 C CNN
 F 3 "~" H 10550 3500 50  0001 C CNN
 	1    10550 3500
@@
 F 0 "D7" V 7796 4471 50  0000 R CNN
 F 1 "D_Sch" V 7705 4471 50  0000 R CNN
-F 2 "Diode_THT:D_DO-27_P5.08mm_Vertical_AnodeUp" H 7750 4550 50  0001 C CNN
+F 2 "Diode_SMD:D_SOT-23_ANK" H 7750 4550 50  0001 C CNN
 F 3 "~" H 7750 4550 50  0001 C CNN
 	1    7750 4550
@@
 F 0 "D6" V 7246 4871 50  0000 R CNN
 F 1 "D_Sch" V 7155 4871 50  0000 R CNN
-F 2 "Diode_THT:D_DO-27_P5.08mm_Vertical_AnodeUp" H 7200 4950 50  0001 C CNN
+F 2 "Diode_SMD:D_SOT-23_ANK" H 7200 4950 50  0001 C CNN
 F 3 "~" H 7200 4950 50  0001 C CNN
 	1    7200 4950
@@
 F 0 "D4" V 6546 5471 50  0000 R CNN
 F 1 "D_Sch" V 6455 5471 50  0000 R CNN
-F 2 "Diode_THT:D_DO-27_P5.08mm_Vertical_AnodeUp" H 6500 5550 50  0001 C CNN
+F 2 "Diode_SMD:D_SOT-23_ANK" H 6500 5550 50  0001 C CNN
 F 3 "~" H 6500 5550 50  0001 C CNN
 	1    6500 5550
@@
 F 0 "D10" H 8100 5866 50  0000 C CNN
 F 1 "D_Sch" H 8100 5775 50  0000 C CNN
-F 2 "Diode_THT:D_DO-27_P5.08mm_Vertical_AnodeUp" H 8100 5650 50  0001 C CNN
+F 2 "Diode_SMD:D_SOT-23_ANK" H 8100 5650 50  0001 C CNN
 F 3 "~" H 8100 5650 50  0001 C CNN
 	1    8100 5650
@@
 F 0 "Q24" V 9728 6000 50  0000 C CNN
 F 1 "Q-PNP" V 9637 6000 50  0000 C CNN
-F 2 "Package_TO_SOT_THT:TO-3P-3_Horizontal_TabDown" H 9600 6100 50  0001 C CNN
+F 2 "Package_TO_SOT_SMD:SOT-23_Handsoldering" H 9600 6100 50  0001 C CNN
 F 3 "~" H 9400 6000 50  0001 C CNN
 	1    9400 6000
@@
 F 0 "R40" H 10020 3946 50  0000 L CNN
 F 1 "R" H 10020 3855 50  0000 L CNN
-F 2 "Resistor_SMD:R_0805_2012Metric_Pad1.15x1.40mm_HandSolder" V 9880 3900 50  0001 C CNN
+F 2 "Resistor_THT:R_Axial_Power_L25.0mm_W9.0mm_P30.48mm" V 9880 3900 50  0001 C CNN
 F 3 "~" H 9950 3900 50  0001 C CNN
 	1    9950 3900
@@
 F 0 "J1" H 542 4735 50  0000 C CNN
 F 1 "Conn" H 542 4644 50  0000 C CNN
-F 2 "Connector:Banana_Jack_2Pin" H 650 4550 50  0001 C CNN
+F 2 "Connector_Audio:Jack_3.5mm_CUI_SJ1-3533NG_Horizontal_CircularHoles" H 650 4550 50  0001 C CNN
 F 3 "~" H 650 4550 50  0001 C CNN
 	1    650  4550
@@
 Wire Wire Line
 	6850 5400 6850 4350
-Connection ~ 9050 1850
-Wire Wire Line
-	9050 1850 9450 1850
 Wire Wire Line
 	7750 5650 7750 5300
@@
 Connection ~ 9950 4500
 Wire Wire Line
-	9050 1850 9050 3500
-Wire Wire Line
 	9650 4050 9650 5800
 Wire Wire Line
@@
 Wire Wire Line
 	9050 3500 9050 5650
-Wire Wire Line
-	9050 1350 9050 1850
 Wire Wire Line
 	5600 4950 5600 4800
@@
 Wire Wire Line
 	5700 4300 5700 4150
+Wire Wire Line
+	8950 1850 9450 1850
+Wire Wire Line
+	9050 1350 9050 3500
 $EndSCHEMATC

Commit message: update pcb
Parts:
- added D11, D12: D_Sch, Diode_SMD:D_SOT-23_ANK, symbol Device:D_Schottky
- added Q28: Q-NPN, Package_TO_SOT_THT:TO-3P-3_Horizontal_TabDown, symbol Device:Q_NPN_BCE
- added Q29: Q_PNP, TO_SOT_Packages_SMD:SOT-23_Handsoldering, symbol Device:Q_PNP_BCE
- added R42, R44: R, Resistors_SMD:R_0805_HandSoldering, symbol Device:R
Connections:
- net at C9.1, Q25.1 (B), R21.2: now also D12.2 (A)
- net at C10.2, D10.1 (K), D9.2 (A)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: now also Q28.3 (E), Q29.3 (E)
- net at Q22.3 (E), Q26.3 (E), R39.1: now also R42.1
- net at C8.2, Q24.1 (B), R22.2: now also D11.1 (K)
- net at Q23.3 (E), Q27.3 (E), R40.2: now also R44.1
- net at Q23.1 (B), R35.2: now also D11.2 (A), Q29.2 (C)
- new net: Q28.1 (B), R42.2
- new net: D12.1 (K), Q28.2 (C)
- new net: Q29.1 (B), R44.2
Changed lines of the file:
@@
 Connection ~ 9050 1050
 Wire Wire Line
-	9050 1050 9250 1050
+	9050 1050 9200 1050
 Connection ~ 9050 750
 Wire Wire Line
@@
 $EndComp
 Wire Wire Line
-	9950 2750 9950 2500
+	9950 2750 9950 2700
 Connection ~ 9950 2500
 $Comp
@@
 	9000 6300 9500 6300
 Connection ~ 9000 6000
-Wire Wire Line
-	9000 6000 9200 6000
 $Comp
 L Device:R R38
@@
 	9650 4050 9650 5800
 Wire Wire Line
-	9950 4050 9950 4500
-Wire Wire Line
 	9950 3050 9950 3500
 Wire Wire Line
@@
 Connection ~ 3200 4550
 Wire Wire Line
-	5700 3500 9050 3500
+	5700 3500 8850 3500
 Wire Wire Line
 	5700 3500 5700 3700
@@
 Wire Wire Line
 	8950 1850 9450 1850
-Wire Wire Line
-	9050 1350 9050 3500
 Connection ~ 3400 2300
 Wire Wire Line
@@
 	1    0    0    1
 $EndComp
+$Comp
+L Device:Q_NPN_BCE Q28
+U 1 1 5D31166D
+P 8950 2700
+F 0 "Q28" H 9141 2746 50  0000 L CNN
+F 1 "Q-NPN" H 9141 2655 50  0000 L CNN
+F 2 "Package_TO_SOT_THT:TO-3P-3_Horizontal_TabDown" H 9150 2800 50  0001 C CNN
+F 3 "~" H 8950 2700 50  0001 C CNN
+	1    8950 2700
+	-1   0    0    -1
+$EndComp
+Wire Wire Line
+	9050 1350 9050 3500
+Wire Wire Line
+	9150 2700 9200 2700
+Wire Wire Line
+	9500 2700 9950 2700
+Connection ~ 9950 2700
+Wire Wire Line
+	9950 2700 9950 2500
+Connection ~ 8850 3500
+Wire Wire Line
+	8850 3500 9050 3500
+$Comp
+L Device:D_Schottky D12
+U 1 1 5D3671D3
+P 9200 1450
+F 0 "D12" V 9246 1371 50  0000 R CNN
+F 1 "D_Sch" V 9155 1371 50  0000 R CNN
+F 2 "Diode_SMD:D_SOT-23_ANK" H 9200 1450 50  0001 C CNN
+F 3 "~" H 9200 1450 50  0001 C CNN
+	1    9200 1450
+	0    -1   -1   0
+$EndComp
+Wire Wire Line
+	8850 2500 8850 2300
+Wire Wire Line
+	8850 2300 9200 2300
+Wire Wire Line
+	9200 2300 9200 1600
+Wire Wire Line
+	9200 1300 9200 1050
+Connection ~ 9200 1050
+Wire Wire Line
+	9200 1050 9250 1050
+Wire Wire Line
+	9150 4150 9200 4150
+Wire Wire Line
+	9500 4150 9950 4150
+Wire Wire Line
+	9950 4050 9950 4150
+Connection ~ 9950 4150
+Wire Wire Line
+	9950 4150 9950 4500
+Wire Wire Line
+	8850 2900 8850 3500
+Wire Wire Line
+	8850 3950 8850 3500
+$Comp
+L Device:D_Schottky D11
+U 1 1 5D3CC3C7
+P 9150 5550
+F 0 "D11" V 9196 5471 50  0000 R CNN
+F 1 "D_Sch" V 9105 5471 50  0000 R CNN
+F 2 "Diode_SMD:D_SOT-23_ANK" H 9150 5550 50  0001 C CNN
+F 3 "~" H 9150 5550 50  0001 C CNN
+	1    9150 5550
+	0    -1   -1   0
+$EndComp
+$Comp
+L Device:Q_PNP_BCE Q29
+U 1 1 5D388C0F
+P 8950 4150
+F 0 "Q29" H 9140 4104 50  0000 L CNN
+F 1 "Q_PNP" H 9140 4195 50  0000 L CNN
+F 2 "TO_SOT_Packages_SMD:SOT-23_Handsoldering" H 9150 4250 50  0001 C CNN
+F 3 "~" H 8950 4150 50  0001 C CNN
+	1    8950 4150
+	-1   0    0    1
+$EndComp
+$Comp
+L Device:R R44
+U 1 1 5D390252
+P 9350 4150
+F 0 "R44" H 9420 4196 50  0000 L CNN
+F 1 "R" H 9420 4105 50  0000 L CNN
+F 2 "Resistors_SMD:R_0805_HandSoldering" V 9280 4150 50  0001 C CNN
+F 3 "~" H 9350 4150 50  0001 C CNN
+	1    9350 4150
+	0    1    1    0
+$EndComp
+Wire Wire Line
+	9150 5700 9150 6000
+Wire Wire Line
+	9000 6000 9150 6000
+Wire Wire Line
+	9150 6000 9200 6000
+Connection ~ 9150 6000
+Wire Wire Line
+	9150 4500 8850 4500
+Wire Wire Line
+	8850 4500 8850 4350
+Wire Wire Line
+	9150 5400 9150 4800
+Wire Wire Line
+	9150 4800 9150 4500
+Connection ~ 9150 4800
+$Comp
+L Device:R R42
+U 1 1 5D3F187F
+P 9350 2700
+F 0 "R42" H 9420 2746 50  0000 L CNN
+F 1 "R" H 9420 2655 50  0000 L CNN
+F 2 "Resistors_SMD:R_0805_HandSoldering" V 9280 2700 50  0001 C CNN
+F 3 "~" H 9350 2700 50  0001 C CNN
+	1    9350 2700
+	0    1    1    0
+$EndComp
 $EndSCHEMATC
