File: PCB/PCB.sch (KiCad schematic (older format))
At the start: 96 parts, among them J1 Conn, J2 Conn, Q1 Q_NPN_BCE, Q10 Q_NPN, Q11 Q_PNP_BCE, Q12 Q_NPN, Q13 Q_PNP, Q14 Q_PNP_BCE, Q15 Q_PNP_BCE, Q16 Q-NPN, Q17 Q-NPN, Q18 Q-NPN, Q19 Q-PNP, Q2 Q_PNP_BCE, Q20 Q-NPN, Q21 Q-PNP, Q22 Q-NPN, Q23 Q-PNP, Q24 Q-PNP, Q25 Q-NPN, Q26 Q-NPN, Q27 Q-PNP, Q28 Q-NPN, Q29 Q_PNP, Q3 Q_NPN_BCE, Q4 Q_PNP_BCE, Q5 Q_NPN_BCE, Q6 Q_PNP_BCE, Q7 Q_PNP_BCE, Q8 Q_NPN_BCE, Q9 Q_NPN_BCE

Commit message: Update PCB
Parts:
- removed D2: LED_ALT, LED_THT:LED_D5.0mm, symbol Device:LED_ALT
- added R43: R, Resistor_SMD:R_0805_2012Metric_Pad1.15x1.40mm_HandSolder, symbol Device:R
- C2: footprint Capacitor_THT:CP_Axial_L11.0mm_D5.0mm_P18.00mm_Horizontal -> Capacitors_THT:CP_Radial_D10.0mm_P7.50mm
- C5: footprint Capacitor_SMD:C_0603_1608Metric_Pad1.05x0.95mm_HandSolder -> Capacitors_THT:CP_Radial_D5.0mm_P2.00mm
- D11, D12: footprint Diode_SMD:D_SOT-23_ANK -> Diodes_SMD:D_SOT-23_ANK
- J1: footprint Connector_Audio:Jack_3.5mm_CUI_SJ1-3533NG_Horizontal_CircularHoles -> Connectors:PJ320D_3.5mm_Jack
- J2: footprint Connector:JWT_A3963_1x02_P3.96mm_Vertical -> Connectors:GTK2400-V2
- Q22, Q23, Q26, Q27: footprint Package_TO_SOT_THT:TO-3P-3_Horizontal_TabDown -> Package_TO_SOT_THT:TO-3P-3_Vertical
- Q28: footprint Package_TO_SOT_THT:TO-3P-3_Horizontal_TabDown -> Package_TO_SOT_SMD:SOT-23_Handsoldering
- Q29: footprint TO_SOT_Packages_SMD:SOT-23_Handsoldering -> Package_TO_SOT_SMD:SOT-23_Handsoldering
- Q8: footprint Package_TO_SOT_THT:TO-3P-3_Horizontal_TabDown -> Package_TO_SOT_THT:TO-126-3_Vertical
- R39, R40: footprint Resistor_THT:R_Axial_Power_L25.0mm_W9.0mm_P30.48mm -> Resistor_THT:R_Axial_Power_L25.0mm_W9.0mm_P7.62mm_Vertical
- R42, R44: footprint Resistors_SMD:R_0805_HandSoldering -> Resistor_SMD:R_0805_2012Metric_Pad1.15x1.40mm_HandSolder
Connections:
- net VEE: now also R43.2
- net at D1.1 (K): now also R43.1
- net at C10.2, D10.1 (K), D9.2 (A)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: now also R39.1; no longer R39.2
- net at Q22.3 (E), Q26.3 (E), R42.1: now also R39.2; no longer R39.1
- net at Q16.2 (C), R35.1: no longer D6.2 (A), R20.2
- net at Q19.2 (C), R17.2: now also D6.2 (A); no longer R20.1
- net at R29.2, R32.2, R36.1: now also R20.2; no longer D6.1 (K)
- new net: D6.1 (K), R20.1
Other:
- moved on the sheet: D6, J1, R20
Changed lines of the file:
@@
 Wire Wire Line
 	1350 6450 1350 6600
-Wire Wire Line
-	3250 7050 3250 6850
 $Comp
 L Device:LED_ALT D1
@@
 	3250 6050 3250 5850
 Connection ~ 3250 5850
-Wire Wire Line
-	3250 6350 3250 6550
 Wire Wire Line
 	1350 5850 1550 5850
@@
 F 0 "C2" H 3085 5054 50  0000 R CNN
 F 1 "C" H 3085 5145 50  0000 R CNN
-F 2 "Capacitor_THT:CP_Axial_L11.0mm_D5.0mm_P18.00mm_Horizontal" H 3238 4950 50  0001 C CNN
+F 2 "Capacitors_THT:CP_Radial_D10.0mm_P7.50mm" H 3238 4950 50  0001 C CNN
 F 3 "~" H 3200 5100 50  0001 C CNN
 	1    3200 5100
@@
 F 0 "Q8" H 4341 3746 50  0000 L CNN
 F 1 "Q_NPN_BCE" H 4341 3655 50  0000 L CNN
-F 2 "Package_TO_SOT_THT:TO-3P-3_Horizontal_TabDown" H 4350 3800 50  0001 C CNN
+F 2 "Package_TO_SOT_THT:TO-126-3_Vertical" H 4350 3800 50  0001 C CNN
 F 3 "~" H 4150 3700 50  0001 C CNN
 	1    4150 3700
@@
 F 0 "C5" H 4485 4254 50  0000 R CNN
 F 1 "C" H 4485 4345 50  0000 R CNN
-F 2 "Capacitor_SMD:C_0603_1608Metric_Pad1.05x0.95mm_HandSolder" H 4638 4150 50  0001 C CNN
+F 2 "Capacitors_THT:CP_Radial_D5.0mm_P2.00mm" H 4638 4150 50  0001 C CNN
 F 3 "~" H 4600 4300 50  0001 C CNN
 	1    4600 4300
@@
 Wire Wire Line
 	4600 5500 4250 5500
-$Comp
-L Device:LED_ALT D2
-U 1 1 5D1D8768
-P 3250 6700
-F 0 "D2" V 3289 6582 50  0000 R CNN
-F 1 "LED_ALT" V 3198 6582 50  0000 R CNN
-F 2 "LED_THT:LED_D5.0mm" H 3250 6700 50  0001 C CNN
-F 3 "~" H 3250 6700 50  0001 C CNN
-	1    3250 6700
-	0    -1   -1   0
-$EndComp
 Wire Wire Line
 	6150 1050 6300 1050
@@
 F 0 "Q26" H 10041 1396 50  0000 L CNN
 F 1 "Q-NPN" H 10041 1305 50  0000 L CNN
-F 2 "Package_TO_SOT_THT:TO-3P-3_Horizontal_TabDown" H 10050 1450 50  0001 C CNN
+F 2 "Package_TO_SOT_THT:TO-3P-3_Vertical" H 10050 1450 50  0001 C CNN
 F 3 "~" H 9850 1350 50  0001 C CNN
 	1    9850 1350
@@
 F 0 "Q22" H 9541 2146 50  0000 L CNN
 F 1 "Q-NPN" H 9541 2055 50  0000 L CNN
-F 2 "Package_TO_SOT_THT:TO-3P-3_Horizontal_TabDown" H 9550 2200 50  0001 C CNN
+F 2 "Package_TO_SOT_THT:TO-3P-3_Vertical" H 9550 2200 50  0001 C CNN
 F 3 "~" H 9350 2100 50  0001 C CNN
 	1    9350 2100
@@
 F 0 "R39" H 10020 2946 50  0000 L CNN
 F 1 "R" H 10020 2855 50  0000 L CNN
-F 2 "Resistor_THT:R_Axial_Power_L25.0mm_W9.0mm_P30.48mm" V 9880 2900 50  0001 C CNN
+F 2 "Resistor_THT:R_Axial_Power_L25.0mm_W9.0mm_P7.62mm_Vertical" V 9880 2900 50  0001 C CNN
 F 3 "~" H 9950 2900 50  0001 C CNN
 	1    9950 2900
-	1    0    0    -1
+	-1   0    0    1
 $EndComp
 Wire Wire Line
@@
 F 0 "J2" H 10578 3476 50  0000 L CNN
 F 1 "Conn" H 10578 3385 50  0000 L CNN
-F 2 "Connector:JWT_A3963_1x02_P3.96mm_Vertical" H 10550 3500 50  0001 C CNN
+F 2 "Connectors:GTK2400-V2" H 10550 3500 50  0001 C CNN
 F 3 "~" H 10550 3500 50  0001 C CNN
 	1    10550 3500
@@
 L Device:D_Schottky D6
 U 1 1 5D3B2CA6
-P 7200 4950
-F 0 "D6" V 7246 4871 50  0000 R CNN
-F 1 "D_Sch" V 7155 4871 50  0000 R CNN
-F 2 "Diode_SMD:D_SOT-23_ANK" H 7200 4950 50  0001 C CNN
-F 3 "~" H 7200 4950 50  0001 C CNN
-	1    7200 4950
+P 7200 4600
+F 0 "D6" V 7246 4521 50  0000 R CNN
+F 1 "D_Sch" V 7155 4521 50  0000 R CNN
+F 2 "Diode_SMD:D_SOT-23_ANK" H 7200 4600 50  0001 C CNN
+F 3 "~" H 7200 4600 50  0001 C CNN
+	1    7200 4600
 	0    -1   -1   0
 $EndComp
@@
 L Device:R R20
 U 1 1 5D3B3972
-P 7200 4600
-F 0 "R20" H 7270 4646 50  0000 L CNN
-F 1 "R" H 7270 4555 50  0000 L CNN
-F 2 "Resistor_SMD:R_0805_2012Metric_Pad1.15x1.40mm_HandSolder" V 7130 4600 50  0001 C CNN
-F 3 "~" H 7200 4600 50  0001 C CNN
-	1    7200 4600
+P 7200 5100
+F 0 "R20" H 7270 5146 50  0000 L CNN
+F 1 "R" H 7270 5055 50  0000 L CNN
+F 2 "Resistor_SMD:R_0805_2012Metric_Pad1.15x1.40mm_HandSolder" V 7130 5100 50  0001 C CNN
+F 3 "~" H 7200 5100 50  0001 C CNN
+	1    7200 5100
 	1    0    0    -1
 $EndComp
@@
 Connection ~ 7200 4350
 Wire Wire Line
-	7200 4750 7200 4800
-Wire Wire Line
-	7200 5100 7200 5450
+	7200 5250 7200 5450
 Wire Wire Line
 	7200 5450 8500 5450
@@
 F 0 "Q27" V 10178 5800 50  0000 C CNN
 F 1 "Q-PNP" V 10087 5800 50  0000 C CNN
-F 2 "Package_TO_SOT_THT:TO-3P-3_Horizontal_TabDown" H 10050 5900 50  0001 C CNN
+F 2 "Package_TO_SOT_THT:TO-3P-3_Vertical" H 10050 5900 50  0001 C CNN
 F 3 "~" H 9850 5800 50  0001 C CNN
 	1    9850 5800
@@
 F 0 "R40" H 10020 3946 50  0000 L CNN
 F 1 "R" H 10020 3855 50  0000 L CNN
-F 2 "Resistor_THT:R_Axial_Power_L25.0mm_W9.0mm_P30.48mm" V 9880 3900 50  0001 C CNN
+F 2 "Resistor_THT:R_Axial_Power_L25.0mm_W9.0mm_P7.62mm_Vertical" V 9880 3900 50  0001 C CNN
 F 3 "~" H 9950 3900 50  0001 C CNN
 	1    9950 3900
@@
 F 0 "Q23" V 9678 4800 50  0000 C CNN
 F 1 "Q-PNP" V 9587 4800 50  0000 C CNN
-F 2 "Package_TO_SOT_THT:TO-3P-3_Horizontal_TabDown" H 9550 4900 50  0001 C CNN
+F 2 "Package_TO_SOT_THT:TO-3P-3_Vertical" H 9550 4900 50  0001 C CNN
 F 3 "~" H 9350 4800 50  0001 C CNN
 	1    9350 4800
@@
 $EndComp
 Wire Wire Line
-	8650 4800 7200 4800
-Connection ~ 7200 4800
-Wire Wire Line
-	7200 4800 6700 4800
-Wire Wire Line
 	8950 4800 9150 4800
 Wire Wire Line
@@
 Wire Wire Line
 	9450 4600 9450 4500
-$Comp
-L Connector:Conn_01x02_Female J1
-U 1 1 5D1D8FF0
-P 650 4550
-F 0 "J1" H 542 4735 50  0000 C CNN
-F 1 "Conn" H 542 4644 50  0000 C CNN
-F 2 "Connector_Audio:Jack_3.5mm_CUI_SJ1-3533NG_Horizontal_CircularHoles" H 650 4550 50  0001 C CNN
-F 3 "~" H 650 4550 50  0001 C CNN
-	1    650  4550
-	-1   0    0    -1
-$EndComp
 Wire Wire Line
 	1300 5250 1300 5150
@@
 	1350 4550 1300 4550
 Connection ~ 1300 4550
-Wire Wire Line
-	850  4550 950  4550
-Wire Wire Line
-	850  4650 950  4650
 Wire Wire Line
 	950  4650 950  5150
@@
 F 0 "Q28" H 9141 2746 50  0000 L CNN
 F 1 "Q-NPN" H 9141 2655 50  0000 L CNN
-F 2 "Package_TO_SOT_THT:TO-3P-3_Horizontal_TabDown" H 9150 2800 50  0001 C CNN
+F 2 "Package_TO_SOT_SMD:SOT-23_Handsoldering" H 9150 2800 50  0001 C CNN
 F 3 "~" H 8950 2700 50  0001 C CNN
 	1    8950 2700
@@
 F 0 "D12" V 9246 1371 50  0000 R CNN
 F 1 "D_Sch" V 9155 1371 50  0000 R CNN
-F 2 "Diode_SMD:D_SOT-23_ANK" H 9200 1450 50  0001 C CNN
+F 2 "Diodes_SMD:D_SOT-23_ANK" H 9200 1450 50  0001 C CNN
 F 3 "~" H 9200 1450 50  0001 C CNN
 	1    9200 1450
@@
 F 0 "D11" V 9196 5471 50  0000 R CNN
 F 1 "D_Sch" V 9105 5471 50  0000 R CNN
-F 2 "Diode_SMD:D_SOT-23_ANK" H 9150 5550 50  0001 C CNN
+F 2 "Diodes_SMD:D_SOT-23_ANK" H 9150 5550 50  0001 C CNN
 F 3 "~" H 9150 5550 50  0001 C CNN
 	1    9150 5550
@@
 F 0 "Q29" H 9140 4104 50  0000 L CNN
 F 1 "Q_PNP" H 9140 4195 50  0000 L CNN
-F 2 "TO_SOT_Packages_SMD:SOT-23_Handsoldering" H 9150 4250 50  0001 C CNN
+F 2 "Package_TO_SOT_SMD:SOT-23_Handsoldering" H 9150 4250 50  0001 C CNN
 F 3 "~" H 8950 4150 50  0001 C CNN
 	1    8950 4150
@@
 F 0 "R44" H 9420 4196 50  0000 L CNN
 F 1 "R" H 9420 4105 50  0000 L CNN
-F 2 "Resistors_SMD:R_0805_HandSoldering" V 9280 4150 50  0001 C CNN
+F 2 "Resistor_SMD:R_0805_2012Metric_Pad1.15x1.40mm_HandSolder" V 9280 4150 50  0001 C CNN
 F 3 "~" H 9350 4150 50  0001 C CNN
 	1    9350 4150
@@
 F 0 "R42" H 9420 2746 50  0000 L CNN
 F 1 "R" H 9420 2655 50  0000 L CNN
-F 2 "Resistors_SMD:R_0805_HandSoldering" V 9280 2700 50  0001 C CNN
+F 2 "Resistor_SMD:R_0805_2012Metric_Pad1.15x1.40mm_HandSolder" V 9280 2700 50  0001 C CNN
 F 3 "~" H 9350 2700 50  0001 C CNN
 	1    9350 2700
@@
 	1    0    0    1
 $EndComp
+Wire Wire Line
+	3250 6350 3250 6550
+$Comp
+L Connector:Conn_01x02_Female J1
+U 1 1 5D1D8FF0
+P 600 4550
+F 0 "J1" H 492 4735 50  0000 C CNN
+F 1 "Conn" H 492 4644 50  0000 C CNN
+F 2 "Connectors:PJ320D_3.5mm_Jack" H 600 4550 50  0001 C CNN
+F 3 "~" H 600 4550 50  0001 C CNN
+	1    600  4550
+	-1   0    0    -1
+$EndComp
+Wire Wire Line
+	800  4550 950  4550
+Wire Wire Line
+	950  4650 800  4650
+$Comp
+L Device:R R43
+U 1 1 5D3BEEE9
+P 3250 6700
+F 0 "R43" H 3320 6746 50  0000 L CNN
+F 1 "R" H 3320 6655 50  0000 L CNN
+F 2 "Resistor_SMD:R_0805_2012Metric_Pad1.15x1.40mm_HandSolder" V 3180 6700 50  0001 C CNN
+F 3 "~" H 3250 6700 50  0001 C CNN
+	1    3250 6700
+	1    0    0    -1
+$EndComp
+Wire Wire Line
+	3250 6850 3250 7050
+Wire Wire Line
+	6700 4800 8650 4800
+Wire Wire Line
+	7200 4750 7200 4950
 $EndSCHEMATC
