File: PCB/PCB.kicad_pcb (KiCad board)
At the start: 2 copper layers, 90 parts, among them J1 Conn, J2 Conn, Q1 Q_NPN_BCE, Q10 Q_NPN, Q11 Q_PNP_BCE, Q12 Q_NPN, Q13 Q_PNP, Q14 Q_PNP_BCE, Q15 Q_PNP_BCE, Q16 Q-NPN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

Commit message: pcb
Parts:
- C2: footprint Capacitor_THT:CP_Axial_L29.0mm_D16.0mm_P35.00mm_Horizontal -> Capacitor_THT:CP_Axial_L11.0mm_D5.0mm_P18.00mm_Horizontal
- D10, D3, D4, D5, D6, D7, D8, D9: footprint Diode_THT:D_DO-27_P5.08mm_Vertical_AnodeUp -> Diode_SMD:D_SOT-23_ANK
- J1: footprint Connector:Banana_Jack_2Pin -> Connector_Audio:Jack_3.5mm_CUI_SJ1-3533NG_Horizontal_CircularHoles
- J2: footprint Connector:Banana_Jack_2Pin -> Connector:JWT_A3963_1x02_P3.96mm_Vertical
- Q24, Q25: footprint Package_TO_SOT_THT:TO-3P-3_Horizontal_TabDown -> Package_TO_SOT_SMD:SOT-23_Handsoldering
- R39, R40: footprint Resistor_SMD:R_0805_2012Metric_Pad1.15x1.40mm_HandSolder -> Resistor_THT:R_Axial_Power_L25.0mm_W9.0mm_P30.48mm
- moved Q23 257.8 mm to (259.1, 129.5), turned to 270 degrees
- moved Q22 240.6 mm to (257.8, 36.8), turned to 270 degrees
- moved J2 224.6 mm to (229.9, 78.7), turned to 270 degrees
- moved Q27 223.5 mm to (259.1, 149.9), turned to 270 degrees
- moved Q8 177.5 mm to (257.8, 69.8), turned to 270 degrees
- moved Q26 177.5 mm to (257.8, 16.5), turned to 270 degrees
- moved R39 174.7 mm to (247.7, 47.0), turned to 270 degrees
- moved R37 152.1 mm to (226.1, 93.0), turned to 270 degrees
- moved R40 143.2 mm to (247.7, 99.1), turned to 270 degrees
- moved Q15 126.2 mm to (58.4, 149.9)
- moved R38 111.3 mm to (219.7, 99.3), turned to 270 degrees
- moved R32 43.8 mm to (130.8, 97.8)
- moved C10 43.5 mm to (92.7, 24.1)
- moved R25 42.3 mm to (83.8, 114.3)
- moved R21 42.1 mm to (108.2, 119.4)
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Connections:
- C10 pad 2: +15V -> Net-(C10-Pad2)
- D10 pad 1: +15V -> Net-(C10-Pad2)
- D9 pad 2: +15V -> Net-(C10-Pad2)
- J2 pad 1: +15V -> Net-(C10-Pad2)
- R37 pad 2: +15V -> Net-(C10-Pad2)
- R38 pad 1: +15V -> Net-(C10-Pad2)
- R39 pad 2: +15V -> Net-(C10-Pad2)
- R40 pad 1: +15V -> Net-(C10-Pad2)
- R41 pad 1: +15V -> Net-(C10-Pad2)

Commit message: Update
Parts:
- C2: footprint Capacitor_THT:CP_Axial_L11.0mm_D5.0mm_P18.00mm_Horizontal -> Capacitor_THT:CP_Radial_D8.0mm_P5.00mm
- Q22, Q23, Q26, Q27: footprint Package_TO_SOT_THT:TO-3P-3_Horizontal_TabDown -> Package_TO_SOT_THT:TO-3P-3_Vertical
- Q24, Q25: footprint Package_TO_SOT_SMD:SOT-23_Handsoldering -> Package_TO_SOT_THT:TO-126-3_Vertical
- Q8: footprint Package_TO_SOT_THT:TO-3P-3_Horizontal_TabDown -> Package_TO_SOT_THT:TO-126-3_Vertical
- R39, R40: footprint Resistor_THT:R_Axial_Power_L25.0mm_W9.0mm_P30.48mm -> Resistor_THT:R_Axial_Power_L25.0mm_W9.0mm_P10.16mm_Vertical
- moved C8 240.1 mm to (256.4, 121.1), turned to 180 degrees
- moved C9 229.0 mm to (242.5, 39.0)
- moved Q15 214.5 mm to (245.5, 45.0), turned to 180 degrees
- moved Q9 204.7 mm to (257.0, 113.0)
- moved Q13 201.8 mm to (251.0, 117.0), turned to 180 degrees
- moved Q25 201.4 mm to (264.5, 57.5), turned to 90 degrees
- moved R41 188.0 mm to (211.5, 62.0), turned to 180 degrees
- moved Q11 186.6 mm to (245.0, 114.0), turned to 180 degrees
- moved Q17 182.0 mm to (246.0, 119.5), turned to 90 degrees
- moved R22 181.3 mm to (251.3, 121.1)
- moved D7 181.2 mm to (162.3, 35.2)
- moved Q14 181.1 mm to (239.5, 44.5), turned to 90 degrees
- moved Q7 178.7 mm to (214.0, 80.0), turned to 180 degrees
- moved Q12 174.7 mm to (214.0, 75.5), turned to 180 degrees
- moved R34 172.0 mm to (247.0, 51.5)
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Routing:
- net (no net): track 0.00 -> 468.5 mm
- net Net-(Q23-Pad3): track 0.00 -> 1.71 mm

Commit message: update pcb
Parts:
- added Q29: Q_PNP, TO_SOT_Packages_SMD:SOT-23_Handsoldering, F.Cu at (221.2, 47.5)
- added R42: R, Resistors_SMD:R_0805_HandSoldering, F.Cu at (227.3, 46.7)
- added R44: R, Resistors_SMD:R_0805_HandSoldering, F.Cu at (227.3, 49.5)

Commit message: update pcb
Parts:
- R37: footprint Resistor_SMD:R_0805_2012Metric_Pad1.15x1.40mm_HandSolder -> Resistor_THT:R_Axial_DIN0207_L6.3mm_D2.5mm_P10.16mm_Horizontal
- moved Q9 205.3 mm to (53.5, 140.5)
- moved C8 187.3 mm to (69.3, 131.1)
- moved Q11 187.3 mm to (58.0, 124.0)
- moved Q13 187.3 mm to (64.0, 127.0)
- moved Q17 187.3 mm to (59.0, 129.5)
- moved R12 187.3 mm to (53.5, 124.0)
- moved R14 187.3 mm to (64.5, 123.0)
- moved R22 187.3 mm to (64.3, 131.1)
- moved R38 187.3 mm to (71.5, 134.5)
- moved R25 146.6 mm to (58.5, 100.5)
- moved R26 146.6 mm to (58.5, 103.5)
- moved R27 146.6 mm to (58.5, 97.5)
- moved Q29 139.1 mm to (83.0, 31.0)
- moved R17 138.7 mm to (61.0, 49.5)
- moved Q20 138.5 mm to (55.5, 42.0)
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Routing:
- net (no net): track 468.5 -> 0.00 mm
- net VCC: track 0.00 -> 421.7 mm, vias 0 -> 1
- net VEE: track 0.00 -> 338.5 mm
- net +15V: track 0.00 -> 321.9 mm
- net -15V: track 0.00 -> 307.4 mm
- net Net-(Q12-Pad3): track 0.00 -> 71.1 mm
- net Net-(C10-Pad2): track 0.00 -> 70.9 mm
- net Net-(Q23-Pad3): track 1.71 -> 45.0 mm
- net Net-(Q22-Pad1): track 0.00 -> 33.3 mm
- net Net-(D5-Pad2): track 0.00 -> 32.2 mm
- net Net-(Q22-Pad3): track 0.00 -> 31.7 mm
- net Net-(Q25-Pad3): track 0.00 -> 29.2 mm
- net Net-(C9-Pad1): track 0.00 -> 26.8 mm
- net Net-(D3-Pad2): track 0.00 -> 24.6 mm
- net Net-(R19-Pad1): track 0.00 -> 19.1 mm
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
Commit message: update pcb
Parts:
- moved Q23 20.5 mm to (272.5, 110.0)
- moved Q27 16.5 mm to (272.5, 90.5)
Routing:
- net Net-(Q23-Pad3): track 45.0 -> 0.00 mm
- net VEE: track 338.5 -> 298.2 mm
- net -15V: track 307.4 -> 283.3 mm
Changed lines of the file:
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@@
     (thickness 1.6)
     (drawings 0)
-    (tracks 145)
+    (tracks 136)
     (zones 0)
     (modules 93)
@@
   )
   (module Package_TO_SOT_THT:TO-3P-3_Vertical (layer F.Cu)
-    (at 272.5 89.5 270)
+    (at 272.5 110.05 270)
     (descr "TO-3P-3, Vertical, RM 5.45mm, , see https://toshiba.semicon-storage.com/ap-en/design-support/package/detail.TO-3P(N).html")
     (tags "TO-3P-3 Vertical RM 5.45mm ")
@@
   )
   (module Package_TO_SOT_THT:TO-3P-3_Vertical (layer F.Cu)
-    (at 272.5 107 270)
+    (at 272.5 90.55 270)
     (descr "TO-3P-3, Vertical, RM 5.45mm, , see https://toshiba.semicon-storage.com/ap-en/design-support/package/detail.TO-3P(N).html")
     (tags "TO-3P-3 Vertical RM 5.45mm ")
@@
   (segment (start 230.4875 66.5) (end 227.4875 69.5) (width 0.25) (layer F.Cu) (net 13))
   (segment (start 231.5 66.5) (end 230.4875 66.5) (width 0.25) (layer F.Cu) (net 13))
-  (segment (start 272.5 113.95) (end 272.5 112.45) (width 0.25) (layer F.Cu) (net 14))
   (segment (start 261 121) (end 260.89 121.11) (width 0.25) (layer F.Cu) (net 14))
-  (segment (start 275 112.45) (end 278 115.45) (width 0.25) (layer B.Cu) (net 14))
-  (segment (start 272.5 112.45) (end 275 112.45) (width 0.25) (layer B.Cu) (net 14))
-  (segment (start 278 115.45) (end 278 147.5) (width 0.25) (layer B.Cu) (net 14))
   (segment (start 278 147.5) (end 267.5 158) (width 0.25) (layer B.Cu) (net 14))
   (segment (start 267.5 158) (end 27.5 158) (width 0.25) (layer B.Cu) (net 14))
@@
   (segment (start 272.5 64.9) (end 263.16 74.24) (width 0.25) (layer F.Cu) (net 58))
   (segment (start 272.5 63.4) (end 272.5 64.9) (width 0.25) (layer F.Cu) (net 58))
-  (segment (start 272.5 94.95) (end 275 94.95) (width 0.25) (layer F.Cu) (net 59))
-  (segment (start 272.5 94.95) (end 270 94.95) (width 0.25) (layer B.Cu) (net 59))
-  (segment (start 275 94.95) (end 279.5 99.45) (width 0.25) (layer F.Cu) (net 59))
-  (segment (start 279.5 99.45) (end 279.5 146) (width 0.25) (layer F.Cu) (net 59))
-  (segment (start 279.5 146) (end 267.5 158) (width 0.25) (layer F.Cu) (net 59))
   (segment (start 267.5 158) (end 35 158) (width 0.25) (layer F.Cu) (net 59))
-  (segment (start 272.5 99.84) (end 272.5 100.4) (width 0.25) (layer F.Cu) (net 60))
-  (segment (start 263.16 90.5) (end 272.5 99.84) (width 0.25) (layer F.Cu) (net 60))
-  (segment (start 272.5 116.4) (end 272.5 117.9) (width 0.25) (layer B.Cu) (net 60))
-  (segment (start 263.16 107.06) (end 272.5 116.4) (width 0.25) (layer B.Cu) (net 60))
-  (segment (start 263.16 90.5) (end 263.16 107.06) (width 0.25) (layer B.Cu) (net 60))
+  (segment (start 272.5 117) (end 272.5 115.5) (width 0.25) (layer F.Cu) (net 59))
+  (segment (start 278.75 123.25) (end 272.5 117) (width 0.25) (layer F.Cu) (net 59))
+  (segment (start 278.75 146.75) (end 278.75 123.25) (width 0.25) (layer F.Cu) (net 59))
+  (segment (start 278.75 146.75) (end 267.5 158) (width 0.25) (layer F.Cu) (net 59))
+  (segment (start 279.5 146) (end 278.75 146.75) (width 0.25) (layer F.Cu) (net 59))
   (segment (start 264.5 52.42) (end 267.5 55.42) (width 0.25) (layer B.Cu) (net 62))
   (segment (start 272.5 70.5) (end 272.5 72) (width 0.25) (layer B.Cu) (net 62))

Commit message: Update PCB
Parts:
- removed D2: LED_ALT, LED_THT:LED_D5.0mm
- added D11: D_Sch, Diodes_SMD:D_SOT-23_ANK, F.Cu at (253.0, 108.7)
- added D12: D_Sch, Diodes_SMD:D_SOT-23_ANK, F.Cu at (252.1, 62.5)
- added Q28: Q-NPN, Package_TO_SOT_SMD:SOT-23_Handsoldering, F.Cu at (253.0, 68.3)
- added R43: R, Resistor_SMD:R_0805_2012Metric_Pad1.15x1.40mm_HandSolder, F.Cu at (148.3, 128.5)
- C2: footprint Capacitor_THT:CP_Radial_D8.0mm_P5.00mm -> Capacitors_THT:CP_Radial_D10.0mm_P7.50mm
- C5: footprint Capacitor_SMD:C_0603_1608Metric_Pad1.05x0.95mm_HandSolder -> Capacitors_THT:CP_Radial_D5.0mm_P2.00mm
- Q24, Q25: footprint Package_TO_SOT_THT:TO-126-3_Vertical -> Package_TO_SOT_SMD:SOT-23_Handsoldering
- Q29: footprint TO_SOT_Packages_SMD:SOT-23_Handsoldering -> Package_TO_SOT_SMD:SOT-23_Handsoldering
- R37: footprint Resistor_THT:R_Axial_DIN0207_L6.3mm_D2.5mm_P10.16mm_Horizontal -> Resistor_SMD:R_0805_2012Metric_Pad1.15x1.40mm_HandSolder
- R39, R40: footprint Resistor_THT:R_Axial_Power_L25.0mm_W9.0mm_P10.16mm_Vertical -> Resistor_THT:R_Axial_Power_L25.0mm_W9.0mm_P7.62mm_Vertical
- R42, R44: footprint Resistors_SMD:R_0805_HandSoldering -> Resistor_SMD:R_0805_2012Metric_Pad1.15x1.40mm_HandSolder
- moved R31 204.1 mm to (245.8, 70.6), turned to 270 degrees
- moved C8 195.1 mm to (263.9, 117.3)
- moved R20 194.4 mm to (224.5, 118.4)
- moved R38 194.2 mm to (262.6, 100.3), turned to 0 degrees
- moved Q20 192.6 mm to (239.0, 100.3)
- moved R22 188.5 mm to (252.0, 113.3)
- moved Q29 184.2 mm to (253.0, 101.9), turned to 90 degrees
- moved R29 181.7 mm to (240.3, 111.3)
- moved R44 178.7 mm to (262.6, 104.9), turned to 180 degrees
- moved R42 170.2 mm to (262.9, 65.0), turned to 180 degrees
- moved R26 168.4 mm to (226.8, 109.0), turned to 0 degrees
- moved Q17 162.0 mm to (221.0, 125.7), turned to 0 degrees
- moved C6 161.9 mm to (226.6, 102.1), turned to 180 degrees
- moved R25 161.5 mm to (219.7, 109.0)
- moved R27 161.4 mm to (219.7, 105.2)
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Connections:
- Q16 pad 2: Net-(D6-Pad2) -> Net-(Q16-Pad2)
- Q19 pad 2: Net-(Q19-Pad2) -> Net-(D6-Pad2)
- R17 pad 2: Net-(Q19-Pad2) -> Net-(D6-Pad2)
- R20 pad 1: Net-(Q19-Pad2) -> Net-(D6-Pad1)
- R20 pad 2: Net-(D6-Pad2) -> Net-(R20-Pad2)
- R29 pad 2: Net-(D6-Pad1) -> Net-(R20-Pad2)
- R32 pad 2: Net-(D6-Pad1) -> Net-(R20-Pad2)
- R35 pad 1: Net-(D6-Pad2) -> Net-(Q16-Pad2)
- R36 pad 1: Net-(D6-Pad1) -> Net-(R20-Pad2)
- R39 pad 1: Net-(Q22-Pad3) -> Net-(C10-Pad2)
- R39 pad 2: Net-(C10-Pad2) -> Net-(Q22-Pad3)
Routing:
- net -15V: track 283.3 -> 0.00 mm
- net VEE: track 298.2 -> 35.1 mm
- net VCC: track 421.7 -> 321.6 mm
- net +15V: track 321.9 -> 260.1 mm
- net Net-(Q23-Pad3): track 0.00 -> 53.6 mm
- net Net-(Q24-Pad3): track 0.00 -> 32.1 mm
- net GND: track 0.00 -> 31.2 mm
- net Net-(D5-Pad2): track 32.2 -> 5.35 mm
- net Net-(Q22-Pad1): track 33.3 -> 8.82 mm
- net Net-(D5-Pad1): track 10.6 -> 28.0 mm
- net Net-(D3-Pad2): track 24.6 -> 7.33 mm
- net Net-(Q22-Pad3): track 31.7 -> 48.6 mm
- net Net-(Q12-Pad3): track 71.1 -> 57.3 mm
- net Net-(C9-Pad1): track 26.8 -> 14.2 mm
- net Net-(C10-Pad2): track 70.9 -> 61.4 mm
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Other:
- net class Default: trace_width 0.25 -> 0.3
- net class Potencia added: clearance 0.3, trace_width 1.5, via_dia 1, via_drill 0.6

Commit message: Etapa salida PCB cheta
Parts:
- moved D4 37.1 mm to (244.1, 118.6)
- moved R17 33.9 mm to (240.4, 116.3)
- moved Q19 32.3 mm to (244.4, 110.6), turned to 270 degrees
- moved Q17 30.2 mm to (250.5, 119.5)
- moved Q13 23.3 mm to (224.3, 119.2)
- moved Q11 22.8 mm to (216.6, 116.8)
- moved D6 22.7 mm to (235.3, 116.3), turned to 180 degrees
- moved R25 19.3 mm to (239.0, 110.6), turned to 90 degrees
- moved R27 16.3 mm to (235.1, 110.5), turned to 90 degrees
- moved Q16 14.9 mm to (258.1, 119.5)
- moved R26 14.2 mm to (239.9, 103.4), turned to 90 degrees
- moved R35 14.1 mm to (266.7, 119.3)
- moved R29 9.81 mm to (230.5, 110.5), turned to 270 degrees
- moved C6 8.75 mm to (235.2, 103.8), turned to 270 degrees
- moved R20 6.70 mm to (230.5, 115.3), turned to 90 degrees
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Routing:
- net VCC: track 321.6 -> 15.8 mm
- net +15V: track 260.1 -> 0.00 mm
- net Net-(D11-Pad2): track 0.00 -> 37.9 mm
- net Net-(Q13-Pad3): track 0.00 -> 33.5 mm
- net Net-(Q16-Pad1): track 0.00 -> 23.3 mm
- net Net-(Q19-Pad3): track 0.00 -> 21.6 mm
- net VEE: track 35.1 -> 13.5 mm
- net Net-(C10-Pad2): track 61.4 -> 80.6 mm
- net Net-(Q20-Pad1): track 0.00 -> 19.0 mm
- net Net-(Q19-Pad1): track 0.00 -> 14.8 mm
- net Net-(D6-Pad2): track 0.00 -> 12.9 mm
- net Net-(C8-Pad2): track 0.00 -> 12.4 mm
- net Net-(C6-Pad1): track 0.00 -> 11.3 mm
- net Net-(R20-Pad2): track 0.00 -> 7.12 mm
- net Net-(Q16-Pad2): track 0.00 -> 6.41 mm
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Other:
- rule trace_min: 0.2 -> 0.3
- rule via_min_size: 0.4 -> 0.3

Commit message: Update PCB
Parts:
- moved C10 66.8 mm to (180.8, 101.9)
- moved R41 66.0 mm to (180.7, 105.7)
- moved R2 61.4 mm to (208.6, 111.2)
- moved R5 61.2 mm to (208.6, 115.8)
- moved Q5 58.6 mm to (175.4, 103.4)
- moved Q4 58.4 mm to (175.4, 95.0)
- moved R8 58.3 mm to (175.4, 110.1)
- moved R7 57.8 mm to (175.6, 68.0)
- moved C2 55.0 mm to (183.6, 85.5)
- moved R3 54.7 mm to (192.2, 91.1)
- moved R9 53.9 mm to (181.9, 92.1)
- moved R12 49.8 mm to (205.9, 85.4)
- moved Q8 48.4 mm to (212.4, 88.1)
- moved R1 47.4 mm to (193.4, 109.8)
- moved R11 47.2 mm to (205.9, 80.9)
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Routing:
- net GND: track 31.2 -> 78.1 mm
- net Net-(D1-Pad2): track 0.00 -> 31.2 mm
- net Net-(Q4-Pad3): track 0.00 -> 24.5 mm
- net Net-(C10-Pad1): track 0.00 -> 22.9 mm
- net VEE: track 13.5 -> 34.6 mm
- net VCC: track 15.8 -> 34.0 mm, vias 1 -> 0
- net Net-(Q2-Pad1): track 0.00 -> 16.0 mm
- net Net-(Q3-Pad2): track 0.00 -> 13.5 mm
- net Net-(Q29-Pad1): track 0.00 -> 12.2 mm
- net Net-(C5-Pad1): track 0.00 -> 7.41 mm
- net Net-(C3-Pad1): track 0.00 -> 6.39 mm
- net Net-(Q3-Pad3): track 0.00 -> 4.90 mm
- net Net-(Q5-Pad3): track 0.00 -> 4.19 mm
- net Net-(D10-Pad2): track 0.00 -> 4.13 mm
- net Net-(Q1-Pad3): track 0.00 -> 4.09 mm
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