File: PCB/PCB.kicad_pcb (KiCad board)
At the start: 2 copper layers, 110 x 80 mm, 99 parts, among them J2 Conn, J3 Screw_Terminal_01x02, J4 Screw_Terminal_01x02, J5 Screw_Terminal_01x02, J6 Screw_Terminal_01x02, Q1 Q_NPN_BCE, Q10 Q_NPN, Q11 Q_PNP_BCE, Q12 Q_NPN, Q13 Q_PNP, Q14 Q_PNP_BCE, Q15 Q_PNP_BCE, Q16 Q-NPN, Q17 Q-NPN, Q18 Q-NPN, Q19 Q-PNP, Q2 Q_PNP_BCE, Q20 Q-NPN, Q21 Q-PNP, Q22 Q-NPN, Q23 Q-PNP, Q24 Q-PNP, Q25 Q-NPN, Q26 Q-NPN, Q27 Q-PNP, Q28 Q-NPN, Q29 Q_PNP, Q3 Q_NPN_BCE, Q4 Q_PNP_BCE, Q5 Q_NPN_BCE, Q6 Q_PNP_BCE, Q7 Q_PNP_BCE, Q8 Q_NPN_BCE, Q9 Q_NPN_BCE

Commit message: update pcb
Parts:
- added REF**: MountingHole_3.5mm, Mounting_Holes:MountingHole_3.5mm, F.Cu at (264.6, 84.6)
- added REF**: MountingHole_3.5mm, Mounting_Holes:MountingHole_3.5mm, F.Cu at (210.0, 94.0)
- added REF**: MountingHole_3.5mm, Mounting_Holes:MountingHole_3.5mm, F.Cu at (276.0, 54.0)
- added REF**: MountingHole_3.5mm, Mounting_Holes:MountingHole_3.5mm, F.Cu at (276.0, 126.0)
- added REF**: MountingHole_3.5mm, Mounting_Holes:MountingHole_3.5mm, F.Cu at (174.0, 126.0)
- added REF**: MountingHole_3.5mm, Mounting_Holes:MountingHole_3.5mm, F.Cu at (174.0, 54.0)
Routing:
- net GND: track 251.7 -> 254.1 mm
- net Net-(C3-Pad2): track 75.2 -> 77.3 mm

Commit message: update pcb
Routing:
- net Net-(Q8-Pad1): track 13.4 -> 12.1 mm
- net Net-(C5-Pad1): track 71.7 -> 71.0 mm

Commit message: update pcb
Parts:
- removed Q2: Q_PNP_BCE, Package_TO_SOT_SMD:SOT-23_Handsoldering
- added REF**: Heatsink_Stonecold_HS-132_32x14mm_2xFixation1.5mm, Heatsinks:Heatsink_Stonecold_HS-132_32x14mm_2xFixation1.5mm, F.Cu at (266.0, 105.5)
- added REF**: Heatsink_Stonecold_HS-132_32x14mm_2xFixation1.5mm, Heatsinks:Heatsink_Stonecold_HS-132_32x14mm_2xFixation1.5mm, F.Cu at (266.0, 70.0)
- C2: footprint Capacitors_THT:CP_Radial_D10.0mm_P7.50mm -> Capacitors_THT:CP_Radial_D10.0mm_P3.80mm
Routing:
- net Net-(C2-Pad2): track 16.1 -> 13.7 mm
